Commit message: Renamed 2130 to 2141

File: ROS/bpl_alpha_description/urdf/RA_2141.urdf.xacro (robot description, xacro)
@@ -1,5 +1,5 @@
 <?xml version="1.0"?>
-<robot name="RA_2130" xmlns:xacro="http://ros.org/wiki/xacro">
-    <xacro:macro name="RA_2130" params="parent *origin name:=RA_2130">
+<robot name="RA_2141" xmlns:xacro="http://ros.org/wiki/xacro">
+    <xacro:macro name="RA_2141" params="parent *origin name:=RA_2141">
         <joint name="${name}_joint" type="fixed">
             <xacro:insert_block name="origin" />
